File: PCB/Monitoring Circuit/V3 - Adding Control Part/v1.brd (EAGLE design)
At the start: 73.3 x 63 mm, 23 parts, among them U1 328P, Y1 16MHz

Commit message: New PCB with control
Parts:
- removed PM25: (no value), SparkFun-Connectors:1X04
- removed POWERINDICATOR: (no value), SparkFun-LED:LED-1206
- removed POWERUSB: USB_B_PTH, SparkFun-Connectors:USB-B-PTH
- removed R5: 1k, SparkFun-Resistors:AXIAL-0.3
- added CONTROL, PM1: (no value), SparkFun-Connectors:1X04
- moved R6 44.2 mm to (58.9, 15.7)
- moved WIFI 44.2 mm to (67.1, 15.7)
- moved R7 44.2 mm to (58.9, 10.2)
- moved SENSORS 44.2 mm to (67.1, 10.2)
- moved MCGS 15.1 mm to (37.6, 43.9)
Connections:
- removed net N$11: U$2.D2, U1.6
- removed net N$15: POWERINDICATOR.A, R5.P$1
- new net N$6: CONTROL.4, U1.26
- net 5V: now also CONTROL.2, PM1.2; no longer PM25.2, POWERUSB.VBUS, R5.P$2
- net GND: now also CONTROL.1, PM1.1; no longer PM25.1, POWERINDICATOR.C, POWERUSB.GND
- net N$8: now also PM1.3; no longer PM25.3
- net N$9: now also PM1.4; no longer PM25.4
Routing:
- net 5V: track 170.0 -> 120.3 mm
- net N$6: track 0.00 -> 47.9 mm
- net GND: track 216.7 -> 178.7 mm, vias 6 -> 4
- net N$8: track 54.1 -> 16.6 mm
- net N$18: track 64.4 -> 27.5 mm, vias 2 -> 0
- net N$16: track 30.5 -> 60.9 mm
- net N$9: track 36.0 -> 13.1 mm
- net N$7: track 42.4 -> 36.9 mm, vias 2 -> 0
- net N$15: track 2.82 -> 0.00 mm, vias 1 -> 0
Other:
- board size 73.3 x 63 mm -> 76.2 x 53.3 mm
