File: PCB/Monitoring Circuit/V3 - Adding Control Part/v1.sch (EAGLE design)
At the start: 23 parts, among them U1 328P, Y1 16MHz

Commit message: New PCB with control
Parts:
- removed PM25: (no value), SparkFun-Connectors:CONN_04
- removed POWERINDICATOR: (no value), SparkFun-LED:LED1206
- removed POWERUSB: USB_B_PTH, SparkFun-Connectors:USB_B_PTH
- removed R5: 1k, SparkFun-Resistors:1KOHM-HORIZ-1/4W-1%
- added CONTROL, PM1: (no value), SparkFun-Connectors:CONN_04
Connections:
- removed net N$11: U$2.D2, U1.PD4(XCK/T0)
- removed net N$15: POWERINDICATOR.A, R5.1
- new net N$6: CONTROL.4, U1.PC3(ADC3)
- net 5V: now also CONTROL.2, PM1.2; no longer PM25.2, POWERUSB.VBUS, R5.2
- net GND: now also CONTROL.1, PM1.1; no longer PM25.1, POWERINDICATOR.C, POWERUSB.GND
- net N$8: now also PM1.3; no longer PM25.3
- net N$9: now also PM1.4; no longer PM25.4
