File: PCB/Control Circuit/V1/schematics.brd (EAGLE design)
At the start: 36.2 x 35.5 mm, 6 parts, among them K1 RELAY-SPDT, Q1 60V/32A/35mΩ

Commit message: Control Circuit v2
Parts:
- removed Q1: 60V/32A/35mΩ, SparkFun-DiscreteSemi:TO220V
- removed R1: 1k, SparkFun-Resistors:AXIAL-0.3
- removed R2: 10k, SparkFun-Resistors:AXIAL-0.3
Connections:
- removed net N$1: Q1.1, R1.P$1, R2.P$1
- removed net N$2: K1.2, Q1.2
- net GND: no longer Q1.3, R2.P$2
- net TRIGGER: no longer R1.P$2
Routing:
- net 5V: track 42.5 -> 0.00 mm
- net N$2: track 22.3 -> 0.00 mm
- net GND: track 16.4 -> 0.00 mm
- net N$1: track 15.0 -> 0.00 mm
- net TRIGGER: track 9.94 -> 0.00 mm
Changed lines of the file:
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@@
 <attribute name="VALUE" x="34.29" y="10.16" size="1.27" layer="27" rot="R90"/>
-</element>
-<element name="Q1" library="SparkFun-DiscreteSemi" package="TO220V" value="60V/32A/35mΩ" x="8.89" y="17.78" smashed="yes" rot="R180">
-<attribute name="NAME" x="14.224" y="17.526" size="0.6096" layer="25" font="vector" ratio="20" rot="R270" align="bottom-center"/>
-<attribute name="PROD_ID" value="TRANS-10060" x="-22.86" y="43.18" size="1.778" layer="27" rot="R180" display="off"/>
-<attribute name="VALUE" x="3.556" y="17.526" size="0.6096" layer="27" font="vector" ratio="20" rot="R270" align="top-center"/>
-</element>
-<element name="R1" library="SparkFun-Resistors" package="AXIAL-0.3" value="1k" x="7.62" y="29.21" smashed="yes" rot="R180">
-<attribute name="NAME" x="7.62" y="28.194" size="0.6096" layer="25" font="vector" ratio="20" rot="R180" align="bottom-center"/>
-<attribute name="PROD_ID" value="RES-12182" x="-10.16" y="62.23" size="1.778" layer="27" rot="R180" display="off"/>
-<attribute name="VALUE" x="7.62" y="30.226" size="0.6096" layer="27" font="vector" ratio="20" rot="R180" align="top-center"/>
-</element>
-<element name="R2" library="SparkFun-Resistors" package="AXIAL-0.3" value="10k" x="7.62" y="31.75" smashed="yes" rot="R180">
-<attribute name="NAME" x="7.62" y="30.734" size="0.6096" layer="25" font="vector" ratio="20" rot="R180" align="bottom-center"/>
-<attribute name="PROD_ID" value="RES-12182" x="-20.32" y="64.77" size="1.778" layer="27" rot="R180" display="off"/>
-<attribute name="VALUE" x="7.62" y="32.766" size="0.6096" layer="27" font="vector" ratio="20" rot="R180" align="top-center"/>
 </element>
 <element name="SIGNAL_IN" library="SparkFun-Connectors" package="1X03" value="" x="10.16" y="24.13" smashed="yes" rot="R180">
@@
 <contactref element="K1" pad="5"/>
 <contactref element="SIGNAL_IN" pad="2"/>
-<wire x1="7.62" y1="24.13" x2="7.62" y2="23.368" width="0.2032" layer="1"/>
-<wire x1="7.62" y1="23.368" x2="8.636" y2="22.352" width="0.2032" layer="1"/>
-<wire x1="8.636" y1="22.352" x2="11.176" y2="22.352" width="0.2032" layer="1"/>
-<wire x1="11.176" y1="22.352" x2="11.938" y2="23.114" width="0.2032" layer="1"/>
-<wire x1="11.938" y1="23.114" x2="11.938" y2="26.162" width="0.2032" layer="1"/>
-<wire x1="11.938" y1="26.162" x2="9.398" y2="28.702" width="0.2032" layer="1"/>
-<wire x1="9.398" y1="28.702" x2="9.398" y2="32.258" width="0.2032" layer="1"/>
-<wire x1="11.5724" y1="34.4324" x2="27.686" y2="34.4324" width="0.2032" layer="1"/>
-<wire x1="27.686" y1="34.4324" x2="30.135" y2="31.9834" width="0.2032" layer="1"/>
-<wire x1="30.135" y1="31.9834" x2="30.135" y2="28.11" width="0.2032" layer="1"/>
-<wire x1="9.398" y1="32.258" x2="11.5724" y2="34.4324" width="0.2032" layer="1"/>
-</signal>
-<signal name="N$2">
-<contactref element="K1" pad="2"/>
-<contactref element="Q1" pad="2"/>
-<wire x1="8.89" y1="17.78" x2="8.89" y2="16.002" width="0.2032" layer="1"/>
-<wire x1="8.89" y1="16.002" x2="9.652" y2="15.24" width="0.2032" layer="1"/>
-<wire x1="9.652" y1="15.24" x2="11.938" y2="15.24" width="0.2032" layer="1"/>
-<wire x1="11.938" y1="15.24" x2="13.208" y2="16.51" width="0.2032" layer="1"/>
-<wire x1="13.208" y1="16.51" x2="13.208" y2="26.162" width="0.2032" layer="1"/>
-<wire x1="13.208" y1="26.162" x2="15.156" y2="28.11" width="0.2032" layer="1"/>
-<wire x1="15.156" y1="28.11" x2="18.135" y2="28.11" width="0.2032" layer="1"/>
+<wire x1="7.62" y1="24.13" x2="30.135" y2="28.11" width="0" layer="19" extent="1-1"/>
 </signal>
 <signal name="GND">
-<contactref element="Q1" pad="3"/>
 <contactref element="SIGNAL_IN" pad="3"/>
-<contactref element="R2" pad="P$2"/>
-<wire x1="6.35" y1="17.78" x2="5.08" y2="19.05" width="0.2032" layer="1"/>
-<wire x1="5.08" y1="19.05" x2="5.08" y2="24.13" width="0.2032" layer="1"/>
-<wire x1="5.08" y1="24.13" x2="2.286" y2="26.924" width="0.2032" layer="1"/>
-<wire x1="2.286" y1="26.924" x2="2.286" y2="30.48" width="0.2032" layer="1"/>
-<wire x1="2.286" y1="30.48" x2="3.556" y2="31.75" width="0.2032" layer="1"/>
-<wire x1="3.556" y1="31.75" x2="3.81" y2="31.75" width="0.2032" layer="1"/>
 </signal>
 <signal name="TRIGGER">
 <contactref element="SIGNAL_IN" pad="1"/>
-<contactref element="R1" pad="P$2"/>
-<wire x1="3.81" y1="29.21" x2="7.62" y2="29.21" width="0.2032" layer="1"/>
-<wire x1="7.62" y1="29.21" x2="10.16" y2="26.67" width="0.2032" layer="1"/>
-<wire x1="10.16" y1="26.67" x2="10.16" y2="24.13" width="0.2032" layer="1"/>
-</signal>
-<signal name="N$1">
-<contactref element="R1" pad="P$1"/>
-<contactref element="Q1" pad="1"/>
-<contactref element="R2" pad="P$1"/>
-<wire x1="11.43" y1="31.75" x2="11.43" y2="29.21" width="0.2032" layer="1"/>
-<wire x1="11.43" y1="17.78" x2="11.43" y2="19.05" width="0.2032" layer="1"/>
-<wire x1="11.43" y1="19.05" x2="12.7" y2="20.32" width="0.2032" layer="1"/>
-<wire x1="12.7" y1="27.94" x2="11.43" y2="29.21" width="0.2032" layer="1"/>
-<wire x1="12.7" y1="20.32" x2="12.7" y2="27.94" width="0.2032" layer="1"/>
 </signal>
 <signal name="N$3">
